Commit message: Restructure workspace: add assem6, assem6_hardware, moveit_config packages and Pi setup docs

File: src/assem6/Assem6/urdf/Assem6.urdf (robot description, URDF)
Before this commit: robot Assem6, 5 links, 4 joints
Links:
- added link world
- link base_link: geometry collision mesh filename=package://assem6/meshes/base_link.STL; visual mesh filename=package://assem6/meshes/base_link.STL
- link link1: geometry collision mesh filename=package://assem6/meshes/link1.STL; visual mesh filename=package://assem6/meshes/link1.STL
- link link2: geometry collision mesh filename=package://assem6/meshes/link2.STL; visual mesh filename=package://assem6/meshes/link2.STL
- link link3: geometry collision mesh filename=package://assem6/meshes/link3.STL; visual mesh filename=package://assem6/meshes/link3.STL
- link link4: geometry collision mesh filename=package://assem6/meshes/link4.STL; visual mesh filename=package://assem6/meshes/link4.STL
Joints:
- added joint world_to_base: type fixed, parent world, child base_link, origin xyz=0 0 0 rpy=0 0 0
